File: pcb/stm32.kicad_sch (KiCad schematic)
At the start: 11 parts, among them U3 STM32F411RETx, Y2 12MHz

Commit message: Preliminary case design done, moving on to PCB design
Parts:
- removed C21, C3: 33p, Capacitor_SMD:C_0805_2012Metric, symbol Device:C_Small
- removed C22: 10n, Capacitor_SMD:C_0603_1608Metric, symbol Device:C
- removed C23: 1u, Capacitor_SMD:C_0603_1608Metric, symbol Device:C
- removed C26: 4.7u, Capacitor_SMD:C_0603_1608Metric, symbol Device:C
- removed C? (x3): 100nF, Capacitor_SMD:C_0603_1608Metric, symbol Device:C_Small
- removed L2: 10u, Inductor_SMD:L_0805_2012Metric, symbol Device:L_Small
- removed U3: STM32F411RETx, Package_QFP:LQFP-64_10x10mm_P0.5mm, symbol MCU_ST_STM32F4:STM32F411RETx
- removed Y2: 12MHz, Crystal:Crystal_SMD_5032-4Pin_5.0x3.2mm, symbol Device:Crystal_GND24
Other:
- note removed: "ADD MORE"
- note removed: "HSE oscillator"
- note removed: "Lowpass LC filter"
- note removed: "MCU protection"
- note removed: "Oscillators"
