File: pcb/keyboard.kicad_sch (KiCad schematic)
At the start: 6 parts

Commit message: Preliminary case design done, moving on to PCB design
Other:
- removed sheet stm32
Changed lines of the file:
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@@
 (kicad_sch (version 20230121) (generator eeschema)
   (paper "A4")
-  (wire (pts (xy 114.3 113.03) (xy 127 113.03))
-    (stroke (width 0) (type default))
-  )
-  (wire (pts (xy 165.1 88.9) (xy 177.8 88.9))
-    (stroke (width 0) (type default))
-  )
-  (wire (pts (xy 114.3 115.57) (xy 127 115.57))
-    (stroke (width 0) (type default))
-  )
-  (wire (pts (xy 114.3 86.36) (xy 127 86.36))
-    (stroke (width 0) (type default))
-  )
-  (wire (pts (xy 114.3 78.74) (xy 127 78.74))
-    (stroke (width 0) (type default))
-  )
-  (wire (pts (xy 114.3 107.95) (xy 127 107.95))
-    (stroke (width 0) (type default))
-  )
-  (wire (pts (xy 114.3 83.82) (xy 127 83.82))
-    (stroke (width 0) (type default))
-  )
-  (wire (pts (xy 114.3 118.11) (xy 127 118.11))
-    (stroke (width 0) (type default))
-  )
-  (wire (pts (xy 114.3 97.79) (xy 127 97.79))
-    (stroke (width 0) (type default))
-  )
-  (wire (pts (xy 114.3 81.28) (xy 127 81.28))
-    (stroke (width 0) (type default))
-  )
-  (wire (pts (xy 114.3 102.87) (xy 127 102.87))
-    (stroke (width 0) (type default))
-  )
-  (wire (pts (xy 114.3 124.46) (xy 127 124.46))
-    (stroke (width 0) (type default))
-  )
-  (wire (pts (xy 114.3 110.49) (xy 127 110.49))
-    (stroke (width 0) (type default))
-  )
-  (wire (pts (xy 114.3 90.17) (xy 127 90.17))
-    (stroke (width 0) (type default))
-  )
-  (wire (pts (xy 165.1 82.55) (xy 177.8 82.55))
-    (stroke (width 0) (type default))
-  )
-  (wire (pts (xy 114.3 121.92) (xy 127 121.92))
-    (stroke (width 0) (type default))
-  )
-  (wire (pts (xy 114.3 92.71) (xy 127 92.71))
-    (stroke (width 0) (type default))
-  )
-  (wire (pts (xy 114.3 95.25) (xy 127 95.25))
-    (stroke (width 0) (type default))
-  )
-  (wire (pts (xy 114.3 100.33) (xy 127 100.33))
-    (stroke (width 0) (type default))
-  )
-  (wire (pts (xy 114.3 105.41) (xy 127 105.41))
-    (stroke (width 0) (type default))
-  )
-  (wire (pts (xy 165.1 80.01) (xy 177.8 80.01))
-    (stroke (width 0) (type default))
-  )
-  (wire (pts (xy 165.1 86.36) (xy 177.8 86.36))
-    (stroke (width 0) (type default))
-  )
   (symbol (lib_id "Mechanical:MountingHole") (at 90.17 154.94 0) (unit 1)
     (in_bom yes) (on_board yes) (dnp no) (fields_autoplaced)
@@
       )
     )
-  )
-  (sheet (at 127 63.5) (size 38.1 76.2) (fields_autoplaced)
-    (stroke (width 0.1524) (type solid))
-    (fill (color 0 0 0 0.0000))
-    (property "Sheetname" "stm32" (at 127 62.7884 0)
-      (effects (font (size 1.27 1.27)) (justify left bottom))
-    )
-    (property "Sheetfile" "stm32.kicad_sch" (at 127 140.2846 0)
-      (effects (font (size 1.27 1.27)) (justify left top))
-    )
-    (property "Field2" "" (at 127 63.5 0)
-      (effects (font (size 1.27 1.27)) hide)
-    )
-    (pin "USB_D-" bidirectional (at 165.1 86.36 0)
-      (effects (font (size 1.27 1.27)) (justify right))
-    )
-    (pin "col6" output (at 127 105.41 180)
-      (effects (font (size 1.27 1.27)) (justify left))
-    )
-    (pin "col8" output (at 127 110.49 180)
-      (effects (font (size 1.27 1.27)) (justify left))
-    )
-    (pin "col7" output (at 127 107.95 180)
-      (effects (font (size 1.27 1.27)) (justify left))
-    )
-    (pin "SWDIO" bidirectional (at 165.1 82.55 0)
-      (effects (font (size 1.27 1.27)) (justify right))
-    )
-    (pin "USB_D+" bidirectional (at 165.1 88.9 0)
-      (effects (font (size 1.27 1.27)) (justify right))
-    )
-    (pin "SWCLK" output (at 165.1 80.01 0)
-      (effects (font (size 1.27 1.27)) (justify right))
-    )
-    (pin "col0" output (at 127 90.17 180)
-      (effects (font (size 1.27 1.27)) (justify left))
-    )
-    (pin "col1" output (at 127 92.71 180)
-      (effects (font (size 1.27 1.27)) (justify left))
-    )
-    (pin "row1" input (at 127 81.28 180)
-      (effects (font (size 1.27 1.27)) (justify left))
-    )
-    (pin "row3" input (at 127 86.36 180)
-      (effects (font (size 1.27 1.27)) (justify left))
-    )
-    (pin "row2" input (at 127 83.82 180)
-      (effects (font (size 1.27 1.27)) (justify left))
-    )
-    (pin "row0" input (at 127 78.74 180)
-      (effects (font (size 1.27 1.27)) (justify left))
-    )
-    (pin "col3" output (at 127 97.79 180)
-      (effects (font (size 1.27 1.27)) (justify left))
-    )
-    (pin "col4" output (at 127 100.33 180)
-      (effects (font (size 1.27 1.27)) (justify left))
-    )
-    (pin "col2" output (at 127 95.25 180)
-      (effects (font (size 1.27 1.27)) (justify left))
-    )
-    (pin "col5" output (at 127 102.87 180)
-      (effects (font (size 1.27 1.27)) (justify left))
-    )
-    (pin "BOOT0" input (at 127 121.92 180)
-      (effects (font (size 1.27 1.27)) (justify left))
-    )
-    (pin "col11" output (at 127 118.11 180)
-      (effects (font (size 1.27 1.27)) (justify left))
-    )
-    (pin "col9" output (at 127 113.03 180)
-      (effects (font (size 1.27 1.27)) (justify left))
-    )
-    (pin "col10" output (at 127 115.57 180)
-      (effects (font (size 1.27 1.27)) (justify left))
-    )
-    (pin "NRST" input (at 127 124.46 180)
-      (effects (font (size 1.27 1.27)) (justify left))
-    )
-    (instances
-      (project "keyboard"
-        (path "/fc529d87-72d0-4c92-b352-ddcf4c6f7199" (page "5"))
-      )
-    )

Commit message: PCB work in progress
Other:
- added sheet MCU (MCU.kicad_sch)
Changed lines of the file:
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@@
+    )
+  )
+  (sheet (at 128.27 69.85) (size 36.83 55.88) (fields_autoplaced)
+    (stroke (width 0.1524) (type solid))
+    (fill (color 0 0 0 0.0000))
+    (property "Sheetname" "MCU" (at 128.27 69.1384 0)
+      (effects (font (size 1.27 1.27)) (justify left bottom))
+    )
+    (property "Sheetfile" "MCU.kicad_sch" (at 128.27 126.3146 0)
+      (effects (font (size 1.27 1.27)) (justify left top))
+    )
+    (property "Field2" "" (at 128.27 69.85 0)
+      (effects (font (size 1.27 1.27)) hide)
+    )
+    (instances
+      (project "keyboard"
+        (path "/fc529d87-72d0-4c92-b352-ddcf4c6f7199" (page "5"))
+      )
     )
   )
@@
     )
   )
-  (sheet (at 177.8 76.2) (size 17.78 20.32) (fields_autoplaced)
+  (sheet (at 177.8 69.85) (size 17.78 20.32) (fields_autoplaced)
     (stroke (width 0.1524) (type solid))
     (fill (color 0 0 0 0.0000))
-    (property "Sheetname" "connectors" (at 177.8 75.4884 0)
+    (property "Sheetname" "connectors" (at 177.8 69.1384 0)
       (effects (font (size 1.27 1.27)) (justify left bottom))
     )
-    (property "Sheetfile" "connectors.kicad_sch" (at 177.8 97.1046 0)
+    (property "Sheetfile" "connectors.kicad_sch" (at 177.8 90.7546 0)
       (effects (font (size 1.27 1.27)) (justify left top))
     )
-    (property "Field2" "" (at 177.8 76.2 0)
+    (property "Field2" "" (at 177.8 69.85 0)
       (effects (font (size 1.27 1.27)) hide)
     )
-    (pin "SWDIO" bidirectional (at 177.8 82.55 180)
+    (pin "SWDIO" bidirectional (at 177.8 76.2 180)
       (effects (font (size 1.27 1.27)) (justify left))
     )
-    (pin "USB_D-" bidirectional (at 177.8 86.36 180)
+    (pin "USB_D-" bidirectional (at 177.8 80.01 180)
       (effects (font (size 1.27 1.27)) (justify left))
     )
-    (pin "USB_D+" bidirectional (at 177.8 88.9 180)
+    (pin "USB_D+" bidirectional (at 177.8 82.55 180)
       (effects (font (size 1.27 1.27)) (justify left))
     )
-    (pin "SWCLK" input (at 177.8 80.01 180)
+    (pin "SWCLK" input (at 177.8 73.66 180)
       (effects (font (size 1.27 1.27)) (justify left))
     )

Commit message: Schematic done, starting PCB design
Parts:
- removed H1, H2, H3, H4, H5, H6: MountingHole, MountingHole:MountingHole_3.2mm_M3, symbol Mechanical:MountingHole
Other:
- sheet MCU ports: added BOOT, SWCLK, SWDIO, USB_D+, USB_D-, col0, col1, col10, col11, col12, col13, col2, col3, col4, col5, col6, col7, col8, col9, row0, row1, row2, row3; removed none
- sheet inputs ports: added BOOT, col12, col13; removed BOOT0, NRST
