File: pcb/keyboard.kicad_pcb (KiCad board)
At the start: 2 copper layers, 242.5 x 98.2 mm, 131 parts, among them J1 USB_C_Receptacle_USB2.0, J2 Conn_01x04, Q2 BC858, SW1 SW_Push, SW10 SW_Push, SW11 SW_Push, SW12 SW_Push, SW13 SW_Push, SW14 SW_Push, SW15 SW_Push, SW16 SW_Push, SW17 SW_Push, SW18 SW_Push, SW19 SW_Push, SW2 SW_Push, SW20 SW_Push, SW21 SW_Push, SW22 SW_Push, SW23 SW_Push, SW24 SW_Push, SW25 SW_Push, SW26 SW_Push, SW27 SW_Push, SW28 SW_Push, SW29 SW_Push, SW3 SW_Push, SW30 SW_Push, SW31 SW_Push, SW32 SW_Push, SW33 SW_Push, SW34 SW_Push, SW35 SW_Push, SW36 SW_Push, SW37 SW_Push, SW38 SW_Push, SW39 SW_Push, SW4 SW_Push, SW40 SW_Push, SW41 SW_Push, SW42 SW_Push, SW43 TS-1187A-B-A-B, SW5 SW_Push, SW6 SW_Push, SW7 SW_Push, SW8 SW_Push, SW9 SW_Push, U1 LP3993-33B3F, U2 USBLC6-2SC6, U3 STM32F411RETx, Y1 12MHz, Y2 32.768k

Commit message: Haven't backed up in a bit
Parts:
- removed C17: 0.1u, Capacitor_SMD:C_0603_1608Metric
- removed C7, C9: 15p, Capacitor_SMD:C_0805_2012Metric
- removed JP1, JP2: bridge, Jumper:SolderJumper-2_P1.3mm_Open_RoundedPad1.0x1.5mm
- removed Q2: BC858, Package_TO_SOT_SMD:SOT-23
- removed R5, R8: 10.2k, Resistor_SMD:R_0603_1608Metric
- removed R7: 1.91k, Resistor_SMD:R_0603_1608Metric
- removed Y2: 32.768k, Crystal:Crystal_SMD_3215-2Pin_3.2x1.5mm
- added D43: D_Small, Diode_SMD:D_SOD-123, F.Cu at (-31.2, 63.0)
- added D44: D_Small, Diode_SMD:D_SOD-123, F.Cu at (-31.2, 66.4)
- added D45: D_Small, Diode_SMD:D_SOD-123, F.Cu at (-31.2, 69.8)
- added D46: D_Small, Diode_SMD:D_SOD-123, F.Cu at (-31.2, 73.1)
- added D47: D_Small, Diode_SMD:D_SOD-123, F.Cu at (-31.2, 76.5)
- added D48: D_Small, Diode_SMD:D_SOD-123, F.Cu at (-31.2, 79.8)
- added Q8: BC858, Package_TO_SOT_SMD:SOT-23, F.Cu at (-25.9, 56.9)
- added SW44: SW_Push, local-library:SW_PG1350, F.Cu at (63.8, -18.0)
- added SW45: SW_Push, local-library:SW_PG1350, F.Cu at (63.8, -1.85)
- added SW46: SW_Push, local-library:SW_PG1350, F.Cu at (63.8, 14.3)
- added SW47: SW_Push, local-library:SW_PG1350, F.Cu at (63.8, 30.4)
- added SW48: SW_Push, local-library:SW_PG1350, F.Cu at (80.8, 50.8)
- C15, D1, D10, D11, D12, D13, D14, D15, D16, D17, D18, D19, D2, D20, D21, D22, D23, D24, D25, D26, D27, D28, D29, D3, D30, D31, D32, D33, D34, D35, D36, D37, D38, D39, D4, D40, D41, D42, D5, D6, D7, D8, D9, J2, L1: moved to F.Cu
- SW43: value TS-1187A-B-A-B -> SW_Push; footprint Button_Switch_SMD:SW_Push_1P1T_NO_CK_KSC6xxJ -> local-library:SW_PG1350
- moved D42 351.9 mm to (-31.2, 59.7), turned to 0 degrees
- moved D40 348.5 mm to (-37.0, 86.5), turned to 0 degrees
- moved D41 347.0 mm to (-31.2, 56.4), turned to 0 degrees
- moved D39 338.5 mm to (-37.0, 83.2), turned to 0 degrees
- moved H5 334.8 mm to (-37.5, 94.2)
- moved D38 334.4 mm to (-37.0, 79.8), turned to 0 degrees
- moved D37 330.8 mm to (-37.0, 76.5), turned to 0 degrees
- moved D36 322.0 mm to (-37.0, 73.1), turned to 0 degrees
- moved H6 321.2 mm to (-37.5, 102.1)
- moved D35 317.4 mm to (-37.0, 69.8), turned to 0 degrees
- moved D34 313.4 mm to (-37.0, 66.4), turned to 0 degrees
- moved D33 312.4 mm to (-37.0, 63.0), turned to 0 degrees
- moved D32 306.6 mm to (-37.0, 59.7), turned to 0 degrees
- moved D30 302.1 mm to (-42.8, 86.5), turned to 0 degrees
- moved D31 301.3 mm to (-37.0, 56.4), turned to 0 degrees
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Connections:
- C16 pad 1: +3V3 -> +3.3V
- SW1 pad 1: Net-(JP2-B) -> +3.3V
- SW1 pad 2: Net-(JP1-A) -> /inputs/BOOT0
- SW25 pad 2: /inputs/col6 -> /inputs/col8
- SW29 pad 2: /inputs/col7 -> /inputs/col9
- SW33 pad 2: /inputs/col8 -> /inputs/col10
- SW43 pad 1: GND -> Net-(D43-A)
- SW43 pad 2: /inputs/NRST -> /inputs/col12
- TP4 pad 1: +3V3 -> +3.3V
- U1 pad 2: +3V3 -> +3.3V
- U3 pad 7: /inputs/NRST -> /stm32/NRST
Routing:
- net /inputs/row0: track 266.6 -> 0.00 mm, vias 1 -> 0
- net /inputs/row2: track 255.4 -> 0.00 mm, vias 1 -> 0
- net /inputs/row1: track 236.5 -> 0.00 mm, vias 1 -> 0
- net +3V3: track 195.0 -> 0.00 mm, vias 2 -> 0
- net /inputs/row3: track 183.6 -> 0.00 mm, vias 1 -> 0
- net /inputs/col0: track 179.4 -> 0.00 mm, vias 4 -> 0
- net /inputs/col11: track 175.5 -> 0.00 mm
- net /inputs/col1: track 162.0 -> 0.00 mm, vias 2 -> 0
- net /inputs/col10: track 154.1 -> 0.00 mm
- net /inputs/col2: track 139.6 -> 0.00 mm, vias 2 -> 0
- net /inputs/col3: track 138.6 -> 0.00 mm, vias 2 -> 0
- net /inputs/col9: track 134.5 -> 0.00 mm
- net /inputs/col8: track 127.5 -> 0.00 mm
- net /inputs/col4: track 123.2 -> 0.00 mm, vias 2 -> 0
- net /inputs/BOOT0: track 116.7 -> 0.00 mm, vias 1 -> 0
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- removed copper zone on F.Cu, net +3V3
- removed copper zone on F.Cu, net +5V
- removed copper zone on F.Cu, net GND
Other:
- board size 242.5 x 98.2 mm -> 331.1 x 102 mm
- board text removed: "3.3V"
- board text removed: "5V"
- board text removed: "CLK"
- board text removed: "Designed by Jack Bradley"
- board text removed: "GND"
- board text removed: "IO"
- board text removed: "JLCJLCJLCJLC"
- board text removed: "Thingamaboard"
- board text removed: "VBUS"
- board text removed: "v1.0"

Commit message: Schematic done, starting PCB design
Parts:
- removed FB1: FerriteBead_Small, Inductor_SMD:L_0603_1608Metric
- removed H1, H2, H3, H4, H5, H6: MountingHole, MountingHole:MountingHole_3.2mm_M3
- removed J2: Conn_01x04, Connector_PinSocket_2.54mm:PinSocket_1x04_P2.54mm_Horizontal
- removed L1: 10u, Inductor_SMD:L_0805_2012Metric
- removed Q8: BC858, Package_TO_SOT_SMD:SOT-23
- removed TP3, TP4: ~, TestPoint:TestPoint_Pad_D2.0mm
- added C7: 100n, Capacitor_SMD:C_0603_1608Metric_Pad1.08x0.95mm_HandSolder, F.Cu at (238.1, -63.5)
- added C9: 1u, Capacitor_SMD:C_0603_1608Metric_Pad1.08x0.95mm_HandSolder, F.Cu at (238.1, -58.4)
- added D49: D_Small, Diode_SMD:D_SOD-123, F.Cu at (130.8, 52.3)
- added Q1: BC858, Package_TO_SOT_SMD:SOT-23, F.Cu at (140.4, 29.4)
- added R10: 10k, Resistor_SMD:R_0603_1608Metric_Pad0.98x0.95mm_HandSolder, F.Cu at (135.8, 33.5)
- added R11: 1k, Resistor_SMD:R_0603_1608Metric_Pad0.98x0.95mm_HandSolder, F.Cu at (246.8, -63.5)
- added R12: 27, Resistor_SMD:R_0603_1608Metric_Pad0.98x0.95mm_HandSolder, F.Cu at (246.8, -60.9)
- added R13: 27, Resistor_SMD:R_0603_1608Metric_Pad0.98x0.95mm_HandSolder, F.Cu at (246.8, -58.4)
- added R5: 10k, Resistor_SMD:R_0603_1608Metric_Pad0.98x0.95mm_HandSolder, F.Cu at (238.1, -42.1)
- added R6: 10k, Resistor_SMD:R_0603_1608Metric_Pad0.98x0.95mm_HandSolder, F.Cu at (238.1, -39.6)
- added R7: 10k, Resistor_SMD:R_0603_1608Metric_Pad0.98x0.95mm_HandSolder, F.Cu at (238.1, -37.1)
- added R8: 10k, Resistor_SMD:R_0603_1608Metric_Pad0.98x0.95mm_HandSolder, F.Cu at (135.8, 28.4)
- added R9: 1k, Resistor_SMD:R_0603_1608Metric_Pad0.98x0.95mm_HandSolder, F.Cu at (135.8, 30.9)
- added U4: RP2040, Package_DFN_QFN:QFN-56-1EP_7x7mm_P0.4mm_EP3.2x3.2mm, F.Cu at (250.9, -52.5)
- C1: value 10n -> 10u; footprint Capacitor_SMD:C_0603_1608Metric -> Capacitor_SMD:C_0603_1608Metric_Pad1.08x0.95mm_HandSolder
- C10: value 10n -> 100n; footprint Capacitor_SMD:C_0603_1608Metric -> Capacitor_SMD:C_0603_1608Metric_Pad1.08x0.95mm_HandSolder
- C11, C12, C15, C5: value 100nF -> 100n; footprint Capacitor_SMD:C_0603_1608Metric -> Capacitor_SMD:C_0603_1608Metric_Pad1.08x0.95mm_HandSolder
- C13, C16: value 1u -> 100n; footprint Capacitor_SMD:C_0603_1608Metric -> Capacitor_SMD:C_0603_1608Metric_Pad1.08x0.95mm_HandSolder
- C14: value 4.7u -> 100n; footprint Capacitor_SMD:C_0603_1608Metric -> Capacitor_SMD:C_0603_1608Metric_Pad1.08x0.95mm_HandSolder
- C2: value 100n -> 10u; footprint Capacitor_SMD:C_0603_1608Metric -> Capacitor_SMD:C_0603_1608Metric_Pad1.08x0.95mm_HandSolder
- C3: value 10u -> 15p; footprint Capacitor_SMD:C_0805_2012Metric -> Capacitor_SMD:C_0805_2012Metric_Pad1.18x1.45mm_HandSolder
- C4: value 1u -> 15p; footprint Capacitor_SMD:C_0603_1608Metric -> Capacitor_SMD:C_0805_2012Metric_Pad1.18x1.45mm_HandSolder
- C6: value 33p -> 100n; footprint Capacitor_SMD:C_0805_2012Metric -> Capacitor_SMD:C_0603_1608Metric_Pad1.08x0.95mm_HandSolder
- C8: value 33p -> 1u; footprint Capacitor_SMD:C_0805_2012Metric -> Capacitor_SMD:C_0603_1608Metric_Pad1.08x0.95mm_HandSolder
- D1: value D_Small -> NCD0805O1; footprint Diode_SMD:D_SOD-123 -> LED_SMD:LED_0805_2012Metric_Pad1.15x1.40mm_HandSolder
- R1, R2, R3: value 10.2k -> 27; footprint Resistor_SMD:R_0603_1608Metric -> Resistor_SMD:R_0603_1608Metric_Pad0.98x0.95mm_HandSolder
- R4: value 10.2k -> 10k; footprint Resistor_SMD:R_0603_1608Metric -> Resistor_SMD:R_0603_1608Metric_Pad0.98x0.95mm_HandSolder
- TP1, TP2: value ~ -> TestPoint
- U1: value LP3993-33B3F -> NCP1117-3.3_SOT223; footprint Package_TO_SOT_SMD:SOT-23 -> Package_TO_SOT_SMD:SOT-223-3_TabPin2
- U3: value STM32F411RETx -> W25Q128JVS; footprint Package_QFP:LQFP-64_10x10mm_P0.5mm -> Package_SO:SOIC-8_5.23x5.23mm_P1.27mm
- Y1: value 12MHz -> ABM8-272_T3; footprint Crystal:Crystal_SMD_5032-4Pin_5.0x3.2mm -> Crystal:Crystal_SMD_3225-4Pin_3.2x2.5mm_HandSoldering
- moved D1 305.9 mm to (242.6, -16.5)
- moved C16 185.5 mm to (246.8, -66.0)
- moved C4 185.1 mm to (251.3, -59.6)
- moved Y1 183.1 mm to (252.2, -66.9)
- moved C15 182.4 mm to (246.8, -68.5)
- moved C3 182.2 mm to (251.3, -62.6)
- moved C5 177.8 mm to (238.1, -68.5)
- moved C10 174.2 mm to (242.4, -68.5)
- moved C11 174.2 mm to (242.4, -66.0)
- moved C12 174.2 mm to (242.4, -63.5)
- moved C13 174.2 mm to (242.4, -60.9)
- moved C14 174.2 mm to (242.4, -58.4)
- moved TP1 171.2 mm to (242.2, -34.4)
- moved TP2 171.2 mm to (242.2, -30.3)
- moved J1 167.1 mm to (245.5, -39.6)
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Connections:
- net /inputs/col12 renamed /MCU/col12
- net /inputs/col13 renamed /MCU/col13
- C14 pad 1: Net-(U3-VCAP1) -> +3V3
- C15 pad 1: Net-(U3-VDDA) -> +3V3
- C16 pad 1: +3.3V -> +3V3
- C2 pad 1: +5V -> +3V3
- C3 pad 1: +5V -> /MCU/XIN
- C4 pad 1: +5V -> GND
- C4 pad 2: GND -> Net-(C4-Pad2)
- C5 pad 1: +5V -> +3V3
- C6 pad 1: /stm32/HSEO_IN -> +1V1
- C8 pad 1: /stm32/HSEO_OUT -> +1V1
- D1 pad 1: /inputs/row0 -> GND
- D1 pad 2: /inputs/S1_OUT -> Net-(D1-A)
- D10 pad 1: /inputs/row0 -> /MCU/row2
- D11 pad 1: /inputs/row1 -> /MCU/row0
- D12 pad 1: /inputs/row2 -> /MCU/row1
- D13 pad 1: /inputs/row3 -> /MCU/row2
- D14 pad 1: /inputs/row0 -> /MCU/row3
- D15 pad 1: /inputs/row1 -> /MCU/row0
- D16 pad 1: /inputs/row2 -> /MCU/row1
- D17 pad 1: /inputs/row3 -> /MCU/row2
- D18 pad 1: /inputs/row0 -> /MCU/row3
- D19 pad 1: /inputs/row1 -> /MCU/row0
- D2 pad 1: /inputs/row1 -> /MCU/row0
- D2 pad 2: Net-(D2-A) -> /inputs/S1_OUT
- D20 pad 1: /inputs/row2 -> /MCU/row1
- D21 pad 1: /inputs/row3 -> /MCU/row2
- D22 pad 1: /inputs/row0 -> /MCU/row3
- D23 pad 1: /inputs/row1 -> /MCU/row0
- D24 pad 1: /inputs/row2 -> /MCU/row1
- D25 pad 1: /inputs/row3 -> /MCU/row2
- D26 pad 1: /inputs/row0 -> /MCU/row0
- D27 pad 1: /inputs/row1 -> /MCU/row1
- D28 pad 1: /inputs/row2 -> /MCU/row2
- D29 pad 1: /inputs/row3 -> /MCU/row0
- D3 pad 1: /inputs/row2 -> /MCU/row1
- D30 pad 1: /inputs/row0 -> /MCU/row1
- D31 pad 1: /inputs/row1 -> /MCU/row2
- D32 pad 1: /inputs/row2 -> /MCU/row3
- D33 pad 1: /inputs/row3 -> /MCU/row0
- D34 pad 1: /inputs/row0 -> /MCU/row1
- D35 pad 1: /inputs/row1 -> /MCU/row2
- D36 pad 1: /inputs/row2 -> /MCU/row3
- D37 pad 1: /inputs/row0 -> /MCU/row0
- D38 pad 1: /inputs/row1 -> /MCU/row1
- D39 pad 1: /inputs/row2 -> /MCU/row2
- D4 pad 1: /inputs/row0 -> /MCU/row2
- D40 pad 1: /inputs/row0 -> /MCU/row3
- D41 pad 1: /inputs/row1 -> /MCU/row0
- D42 pad 1: /inputs/row2 -> /MCU/row1
- D43 pad 1: /inputs/row0 -> /MCU/row2
- D44 pad 1: /inputs/row1 -> /MCU/row0
- D45 pad 1: /inputs/row2 -> /MCU/row1
- D46 pad 1: /inputs/row0 -> /MCU/row2
- D47 pad 1: /inputs/row1 -> /MCU/row0
- D48 pad 1: /inputs/row2 -> /MCU/row1
- D5 pad 1: /inputs/row1 -> /MCU/row0
- D6 pad 1: /inputs/row2 -> /MCU/row1
- D7 pad 1: /inputs/row0 -> /MCU/row2
- D8 pad 1: /inputs/row1 -> /MCU/row0
- D9 pad 1: /inputs/row2 -> /MCU/row1
- J1 pad S1: GND -> unconnected-(J1-SHIELD-PadS1)
- R1 pad 1: /connectors/CC1 -> +3V3
- R1 pad 2: GND -> Net-(R1-Pad2)
- R2 pad 1: /connectors/CC1 -> Net-(R1-Pad2)
- R2 pad 2: GND -> Net-(R2-Pad2)
- R3 pad 1: /connectors/CC2 -> Net-(R2-Pad2)
- R3 pad 2: GND -> Net-(D1-A)
- R4 pad 1: /connectors/CC2 -> /connectors/CC1
- SW1 pad 1: +3.3V -> GND
- SW1 pad 2: /inputs/BOOT0 -> /MCU/BOOT
- SW10 pad 1: Net-(D10-A) -> Net-(D11-A)
- SW10 pad 2: /inputs/col3 -> /MCU/col3
- SW11 pad 1: Net-(D11-A) -> Net-(D12-A)
- SW11 pad 2: /inputs/col3 -> /MCU/col3
- SW12 pad 1: Net-(D12-A) -> Net-(D13-A)
- SW12 pad 2: /inputs/col3 -> /MCU/col3
- SW13 pad 1: Net-(D13-A) -> Net-(D14-A)
- SW13 pad 2: /inputs/col3 -> /MCU/col3
- SW14 pad 1: Net-(D14-A) -> Net-(D15-A)
- SW14 pad 2: /inputs/col4 -> /MCU/col4
- SW15 pad 1: Net-(D15-A) -> Net-(D16-A)
- SW15 pad 2: /inputs/col4 -> /MCU/col4
- SW16 pad 1: Net-(D16-A) -> Net-(D17-A)
- SW16 pad 2: /inputs/col4 -> /MCU/col4
- SW17 pad 1: Net-(D17-A) -> Net-(D18-A)
- SW17 pad 2: /inputs/col4 -> /MCU/col4
- SW18 pad 1: Net-(D18-A) -> Net-(D19-A)
- SW18 pad 2: /inputs/col5 -> /MCU/col5
- SW19 pad 1: Net-(D19-A) -> Net-(D20-A)
- SW19 pad 2: /inputs/col5 -> /MCU/col5
- SW2 pad 1: Net-(D2-A) -> Net-(D3-A)
- SW2 pad 2: /inputs/col0 -> /MCU/col0
- SW20 pad 1: Net-(D20-A) -> Net-(D21-A)
- SW20 pad 2: /inputs/col5 -> /MCU/col5
- SW21 pad 1: Net-(D21-A) -> Net-(D22-A)
- SW21 pad 2: /inputs/col5 -> /MCU/col5
- SW22 pad 1: Net-(D22-A) -> Net-(D23-A)
- SW22 pad 2: /inputs/col6 -> /MCU/col6
- SW23 pad 1: Net-(D23-A) -> Net-(D24-A)
- SW23 pad 2: /inputs/col6 -> /MCU/col6
- SW24 pad 1: Net-(D24-A) -> Net-(D25-A)
- SW24 pad 2: /inputs/col6 -> /MCU/col6
- SW25 pad 1: Net-(D25-A) -> Net-(D26-A)
- SW25 pad 2: /inputs/col8 -> /MCU/col7
- SW26 pad 1: Net-(D26-A) -> Net-(D27-A)
- SW26 pad 2: /inputs/col7 -> /MCU/col7
- SW27 pad 1: Net-(D27-A) -> Net-(D28-A)
- SW27 pad 2: /inputs/col7 -> /MCU/col7
- SW28 pad 1: Net-(D28-A) -> Net-(D29-A)
- SW28 pad 2: /inputs/col7 -> /MCU/col8
- SW29 pad 1: Net-(D29-A) -> Net-(D30-A)
- SW29 pad 2: /inputs/col9 -> /MCU/col8
- SW3 pad 1: Net-(D3-A) -> Net-(D4-A)
- SW3 pad 2: /inputs/col0 -> /MCU/col0
- SW30 pad 1: Net-(D30-A) -> Net-(D31-A)
- SW30 pad 2: /inputs/col8 -> /MCU/col8
- SW31 pad 1: Net-(D31-A) -> Net-(D32-A)
- SW31 pad 2: /inputs/col8 -> /MCU/col8
- SW32 pad 1: Net-(D32-A) -> Net-(D33-A)
- SW32 pad 2: /inputs/col8 -> /MCU/col9
- SW33 pad 1: Net-(D33-A) -> Net-(D34-A)
- SW33 pad 2: /inputs/col10 -> /MCU/col9
- SW34 pad 1: Net-(D34-A) -> Net-(D35-A)
- SW34 pad 2: /inputs/col9 -> /MCU/col9
- SW35 pad 1: Net-(D35-A) -> Net-(D36-A)
- SW35 pad 2: /inputs/col9 -> /MCU/col9
- SW36 pad 1: Net-(D36-A) -> Net-(D37-A)
- SW36 pad 2: /inputs/col9 -> /MCU/col10
- SW37 pad 1: Net-(D37-A) -> Net-(D38-A)
- SW37 pad 2: /inputs/col10 -> /MCU/col10
- SW38 pad 1: Net-(D38-A) -> Net-(D39-A)
- SW38 pad 2: /inputs/col10 -> /MCU/col10
- SW39 pad 1: Net-(D39-A) -> Net-(D40-A)
- SW39 pad 2: /inputs/col10 -> /MCU/col10
- SW4 pad 1: Net-(D4-A) -> Net-(D5-A)
- SW4 pad 2: /inputs/col1 -> /MCU/col1
- SW40 pad 1: Net-(D40-A) -> Net-(D41-A)
- SW40 pad 2: /inputs/col11 -> /MCU/col11
- SW41 pad 1: Net-(D41-A) -> Net-(D42-A)
- SW41 pad 2: /inputs/col11 -> /MCU/col11
- SW42 pad 1: Net-(D42-A) -> Net-(D43-A)
- SW42 pad 2: /inputs/col11 -> /MCU/col11
- SW43 pad 1: Net-(D43-A) -> Net-(D44-A)
- SW44 pad 1: Net-(D44-A) -> Net-(D45-A)
- SW45 pad 1: Net-(D45-A) -> Net-(D46-A)
- SW46 pad 1: Net-(D46-A) -> Net-(D47-A)
- SW47 pad 1: Net-(D47-A) -> Net-(D48-A)
- SW48 pad 1: Net-(D48-A) -> Net-(D49-A)
- SW5 pad 1: Net-(D5-A) -> Net-(D6-A)
- SW5 pad 2: /inputs/col1 -> /MCU/col1
- SW6 pad 1: Net-(D6-A) -> Net-(D7-A)
- SW6 pad 2: /inputs/col1 -> /MCU/col1
- SW7 pad 1: Net-(D7-A) -> Net-(D8-A)
- SW7 pad 2: /inputs/col2 -> /MCU/col2
- SW8 pad 1: Net-(D8-A) -> Net-(D9-A)
- SW8 pad 2: /inputs/col2 -> /MCU/col2
- SW9 pad 1: Net-(D9-A) -> Net-(D10-A)
- SW9 pad 2: /inputs/col2 -> /MCU/col2
- TP1 pad 1: VBUS -> /MCU/SWDIO
- TP2 pad 1: +5V -> /MCU/SWCLK
- U1 pad 2: +3.3V -> +3V3
- U1 pad 3: +5V -> VBUS
- U2 pad 4: /connectors/USB_D+ -> /MCU/USB_D+
- U2 pad 6: /connectors/USB_D- -> /MCU/USB_D-
- U3 pad 1: +3V3 -> /MCU/BOOT
- U3 pad 2: unconnected-(U3-PC13-Pad2) -> /MCU/QSPI_SD1
- U3 pad 3: /stm32/LSEO_IN -> /MCU/QSPI_SD2
- U3 pad 4: /stm32/LSEO_OUT -> GND
- U3 pad 5: /stm32/HSEO_IN -> /MCU/QSPI_SD0
- U3 pad 6: /stm32/HSEO_OUT -> /MCU/QSPI_SCLK
- U3 pad 7: /stm32/NRST -> /MCU/QSPI_SD3
- U3 pad 8: unconnected-(U3-PC0-Pad8) -> +3V3
- Y1 pad 1: /stm32/HSEO_IN -> /MCU/XIN
- Y1 pad 3: /stm32/HSEO_OUT -> Net-(C4-Pad2)
Other:
- outline, holes or cut-outs redrawn

Commit message: Switches placement done, updated footprints to include model
Parts:
- added D26: D_Small, Diode_SMD:D_SOD-123, F.Cu at (75.2, 31.9)
- added D30: D_Small, Diode_SMD:D_SOD-123, F.Cu at (75.2, 35.2)
- added SW25: SW_Push, local-library:SW_PG1350, F.Cu at (173.2, 176.1)
- added SW29: SW_Push, local-library:SW_PG1350, F.Cu at (251.8, 176.1)
- J1: moved to B.Cu
- moved SW33 243.3 mm to (278.3, 166.4), turned to 12 degrees
- moved SW13 222.5 mm to (109.5, 158.0), turned to -12 degrees
- moved SW41 215.1 mm to (315.4, 158.0), turned to 12 degrees
- moved SW40 211.1 mm to (311.4, 139.4), turned to 12 degrees
- moved SW39 207.0 mm to (307.5, 120.8), turned to 12 degrees
- moved SW47 206.9 mm to (349.6, 136.4), turned to 12 degrees
- moved SW46 202.6 mm to (345.7, 117.8), turned to 12 degrees
- moved SW45 198.3 mm to (341.7, 99.2), turned to 12 degrees
- moved SW21 196.3 mm to (146.6, 166.4), turned to -12 degrees
- moved SW20 193.6 mm to (150.6, 147.8), turned to -12 degrees
- moved SW37 191.9 mm to (297.3, 164.4), turned to 12 degrees
- moved SW28 191.5 mm to (254.5, 145.9), turned to 12 degrees
- moved SW19 191.0 mm to (154.5, 129.2), turned to -12 degrees
- moved SW36 187.8 mm to (293.4, 145.8), turned to 12 degrees
- moved SW27 187.7 mm to (250.6, 127.3), turned to 12 degrees
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- renumbered D26 to D27, D27 to D28, D28 to D29, D29 to D31, D30 to D32, D31 to D33, D32 to D34, D33 to D35, D34 to D36, D35 to D37, D36 to D38, D37 to D39, D38 to D40, D39 to D41, D40 to D42, D41 to D43, D42 to D44, D43 to D45, D44 to D46, D45 to D47, D46 to D48, D47 to D49, D48 to D50, D49 to D51, SW25 to SW26, SW26 to SW27, SW27 to SW28, SW28 to SW30, SW29 to SW31, SW30 to SW32, SW31 to SW33, SW32 to SW34, SW33 to SW35, SW34 to SW36, SW35 to SW37, SW36 to SW38, SW37 to SW39, SW38 to SW40, SW39 to SW41, SW40 to SW42, SW41 to SW43, SW42 to SW44, SW43 to SW45, SW44 to SW46, SW45 to SW47, SW46 to SW48, SW47 to SW49, SW48 to SW50

Commit message: Starting diode placement
Parts:
- D10, D11, D12, D13, D14, D15, D16, D17, D18, D19, D2, D20, D21, D22, D23, D24, D25, D26, D27, D28, D29, D3, D30, D31, D32, D33, D34, D35, D36, D37, D38, D39, D4, D40, D41, D42, D43, D44, D45, D46, D47, D48, D49, D5, D50, D51, D6, D7, D8, D9, Q1, R10, R8, R9: moved to B.Cu
- moved D26 181.5 mm to (177.0, 182.2), turned to 63 degrees
- moved D22 147.9 mm to (152.2, 173.0), turned to 78 degrees
- moved D14 129.7 mm to (115.5, 165.2), turned to 78 degrees
- moved D25 127.5 mm to (176.0, 153.0), turned to 78 degrees
- moved D18 122.0 mm to (133.8, 169.2), turned to 78 degrees
- moved D24 116.1 mm to (180.2, 134.4), turned to 78 degrees
- moved D13 114.7 mm to (119.2, 146.8), turned to 78 degrees
- moved D4 113.3 mm to (62.5, 139.5), turned to 78 degrees
- moved D17 110.0 mm to (137.2, 153.0), turned to 78 degrees
- moved Q1 109.1 mm to (49.2, 89.2), turned to 180 degrees
- moved R10 106.3 mm to (46.0, 90.2), turned to -90 degrees
- moved D23 105.7 mm to (184.0, 115.8), turned to 78 degrees
- moved D21 104.9 mm to (156.2, 154.8), turned to 78 degrees
- moved R8 101.3 mm to (51.2, 84.2)
- moved R9 101.1 mm to (51.2, 86.2), turned to 180 degrees
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
Commit message: Diode placement done
Parts:
- moved D51 311.5 mm to (374.8, 138.0), turned to -78 degrees
- moved D50 305.0 mm to (371.8, 120.2), turned to 102 degrees
- moved D48 298.9 mm to (357.8, 140.0), turned to -78 degrees
- moved D49 297.8 mm to (367.8, 101.8), turned to 102 degrees
- moved D47 290.6 mm to (353.8, 122.0), turned to 102 degrees
- moved D45 285.5 mm to (338.8, 142.0), turned to 102 degrees
- moved D46 283.0 mm to (350.0, 103.5), turned to 102 degrees
- moved D44 276.2 mm to (334.8, 123.5), turned to 102 degrees
- moved D42 263.3 mm to (322.0, 161.8), turned to 102 degrees
- moved D38 256.8 mm to (305.0, 168.0), turned to 102 degrees
- moved D41 255.4 mm to (319.5, 143.8), turned to 102 degrees
- moved D43 253.9 mm to (330.8, 105.0), turned to 102 degrees
- moved D34 249.6 mm to (286.5, 170.5), turned to 102 degrees
- moved D37 246.9 mm to (301.5, 150.0), turned to 102 degrees
- moved D40 246.7 mm to (315.8, 125.0), turned to 102 degrees
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
Commit message: Routing in progress
Parts:
- removed the SW26 at (246.6, 108.7)
- added SW2: SW_Push, local-library:SW_PG1350, F.Cu at (64.2, 97.2)
- C1, C10, C11, C12, C13, C14, C15, C16, C2, C3, C4, C5, C6, C7, C8, C9, D1, R1, R11, R12, R13, R2, R3, R4, R5, R6, R7, TP1, TP2, U1, U2, U3, U4: moved to B.Cu
- Y1: footprint Crystal:Crystal_SMD_3225-4Pin_3.2x2.5mm_HandSoldering -> Crystal:Crystal_SMD_3225-4Pin_3.2x2.5mm; moved to B.Cu
- moved C12 240.8 mm to (213.1, 175.5), turned to 180 degrees
- moved C13 240.8 mm to (213.1, 178.0), turned to 180 degrees
- moved C14 240.8 mm to (213.1, 180.5), turned to 180 degrees
- moved C15 227.6 mm to (210.8, 156.2), turned to -90 degrees
- moved Y1 227.4 mm to (217.0, 157.7), turned to -90 degrees
- moved C16 225.9 mm to (206.2, 156.2), turned to -90 degrees
- moved C6 224.1 mm to (209.2, 156.2), turned to -90 degrees
- moved R11 223.8 mm to (214.5, 158.0), turned to 90 degrees
- moved C4 223.2 mm to (217.0, 161.0), turned to 180 degrees
- moved C3 219.7 mm to (217.0, 154.5)
- moved C11 210.8 mm to (206.2, 141.8), turned to 90 degrees
- moved C10 208.7 mm to (214.0, 138.2), turned to 90 degrees
- moved U4 205.0 mm to (212.5, 148.8), turned to 180 degrees
- moved C8 204.7 mm to (209.2, 141.8), turned to 90 degrees
- moved R12 204.3 mm to (212.5, 140.5), turned to -90 degrees
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- renumbered SW9 to SW10, SW10 to SW11, SW11 to SW12, SW12 to SW13, SW13 to SW14, SW14 to SW15, SW15 to SW16, SW16 to SW17, SW17 to SW18, SW18 to SW19, SW19 to SW20, SW20 to SW21, SW21 to SW22, SW22 to SW23, SW23 to SW24, SW24 to SW25, SW25 to SW26, SW2 to SW3, SW3 to SW4, SW4 to SW5, SW5 to SW6, SW6 to SW7, SW7 to SW8, SW8 to SW9
Connections:
- D2 pad 2: /inputs/S1_OUT -> Net-(D2-A)
- D27 pad 2: Net-(D27-A) -> /inputs/SS_OUT
- Q1 pad 2: /MCU/col0 -> /MCU/col7
- Q1 pad 3: /inputs/S1_OUT -> /inputs/SS_OUT
- R10 pad 1: /inputs/S1_OUT -> /inputs/SS_OUT
- U4 pad 2: /MCU/col0 -> /MCU/col7
- U4 pad 3: /MCU/col1 -> /MCU/col8
- U4 pad 35: /MCU/col7 -> /MCU/col0
- U4 pad 36: /MCU/col8 -> /MCU/col1
- U4 pad 37: /MCU/col9 -> /MCU/col2
- U4 pad 38: /MCU/col10 -> /MCU/col3
- U4 pad 39: /MCU/col11 -> /MCU/col4
- U4 pad 4: /MCU/col2 -> /MCU/col9
- U4 pad 40: /MCU/col12 -> /MCU/col5
- U4 pad 41: /MCU/col13 -> /MCU/col6
- U4 pad 5: /MCU/col3 -> /MCU/col10
- U4 pad 6: /MCU/col4 -> /MCU/col11
- U4 pad 7: /MCU/col5 -> /MCU/col12
- U4 pad 8: /MCU/col6 -> /MCU/col13
Routing:
- net /MCU/BOOT: track 0.00 -> 61.5 mm
- net /MCU/USB_D+: track 0.00 -> 28.6 mm
- net /MCU/USB_D-: track 0.00 -> 28.4 mm
- net /MCU/QSPI_SD1: track 0.00 -> 24.9 mm
- net /MCU/QSPI_SD2: track 0.00 -> 23.1 mm
- net +3V3: track 0.00 -> 19.4 mm
- net VBUS: track 0.00 -> 18.5 mm, vias 0 -> 2
- net /MCU/QSPI_SD3: track 0.00 -> 12.5 mm
- net /MCU/QSPI_SCLK: track 0.00 -> 11.3 mm
- net +1V1: track 0.00 -> 10.8 mm
- net /MCU/QSPI_SD0: track 0.00 -> 10.3 mm
- net /MCU/XIN: track 0.00 -> 7.03 mm
- net Net-(J1-D--PadA7): track 0.00 -> 6.89 mm
- net Net-(J1-D+-PadA6): track 0.00 -> 6.86 mm
- net /connectors/CC1: track 0.00 -> 6.72 mm
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
Commit message: More routing progress
Connections:
- U4 pad 2: /MCU/col7 -> /MCU/col13
- U4 pad 3: /MCU/col8 -> /MCU/col12
- U4 pad 35: /MCU/col0 -> /MCU/col6
- U4 pad 36: /MCU/col1 -> /MCU/col5
- U4 pad 37: /MCU/col2 -> /MCU/col4
- U4 pad 39: /MCU/col4 -> /MCU/col2
- U4 pad 4: /MCU/col9 -> /MCU/col11
- U4 pad 40: /MCU/col5 -> /MCU/col1
- U4 pad 41: /MCU/col6 -> /MCU/col0
- U4 pad 6: /MCU/col11 -> /MCU/col9
- U4 pad 7: /MCU/col12 -> /MCU/col8
- U4 pad 8: /MCU/col13 -> /MCU/col7
Routing:
- net /MCU/col6: track 0.00 -> 70.1 mm
- net /MCU/col8: track 0.00 -> 62.1 mm
- net /MCU/col10: track 0.00 -> 61.9 mm
- net /MCU/col9: track 0.00 -> 61.9 mm
- net /MCU/col5: track 0.00 -> 60.7 mm
- net /MCU/col3: track 0.00 -> 60.7 mm
- net /MCU/col4: track 0.00 -> 60.7 mm
- net /MCU/col7: track 0.00 -> 53.7 mm, vias 0 -> 1
- net /MCU/col11: track 0.00 -> 41.8 mm
- net /MCU/col12: track 0.00 -> 41.6 mm
- net /MCU/col13: track 0.00 -> 41.6 mm
- net /MCU/col2: track 0.00 -> 40.4 mm
- net /MCU/col0: track 0.00 -> 40.4 mm
- net /MCU/col1: track 0.00 -> 40.4 mm
- net /inputs/SS_OUT: track 0.00 -> 5.46 mm
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
Commit message: Further progress on routing
Parts:
- added C17: 100n, Capacitor_SMD:C_0603_1608Metric_Pad1.08x0.95mm_HandSolder, B.Cu at (219.0, 145.0)
- TP1, TP2: moved to F.Cu
- moved C2 50.7 mm to (219.0, 129.5)
- moved U1 44.8 mm to (220.0, 124.0), turned to -90 degrees
- moved C1 42.0 mm to (223.2, 118.5), turned to 0 degrees
- moved C12 31.9 mm to (205.5, 144.5)
- moved C14 31.8 mm to (220.0, 149.5), turned to 0 degrees
- moved C13 27.2 mm to (206.2, 151.8), turned to -90 degrees
- moved TP2 23.7 mm to (216.0, 164.2), turned to 0 degrees
- moved TP1 23.3 mm to (212.5, 164.2), turned to 0 degrees
- moved D1 13.3 mm to (231.0, 89.2), turned to 0 degrees
- moved R1 8.43 mm to (231.0, 84.2), turned to 0 degrees
- moved R2 8.17 mm to (231.0, 85.7)
- moved R3 8.02 mm to (231.0, 87.2), turned to 0 degrees
- moved C15 1.25 mm to (210.8, 157.5)
- moved C6 1.25 mm to (209.2, 157.5)
- moved C10 0.79 mm to (214.8, 138.0)
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Routing:
- net /MCU/row0: track 0.00 -> 136.2 mm
- net /MCU/row2: track 0.00 -> 120.3 mm
- net /MCU/row1: track 0.00 -> 120.3 mm
- net +3V3: track 19.4 -> 102.3 mm, vias 0 -> 5
- net /MCU/row3: track 0.00 -> 68.9 mm
- net +1V1: track 10.8 -> 44.4 mm, vias 0 -> 3
- net /MCU/SWDIO: track 0.00 -> 15.7 mm, vias 0 -> 1
- net /MCU/SWCLK: track 0.00 -> 14.9 mm, vias 0 -> 1
- net VBUS: track 18.5 -> 29.8 mm, vias 2 -> 3
- net Net-(D31-A): track 0.00 -> 8.11 mm
- net Net-(D40-A): track 0.00 -> 8.03 mm
- net Net-(D45-A): track 0.00 -> 8.01 mm
- net Net-(D29-A): track 0.00 -> 8.00 mm
- net Net-(D46-A): track 0.00 -> 7.98 mm
- net Net-(D34-A): track 0.00 -> 7.97 mm
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- added copper zone on B.Cu, net VBUS
