File: pcb/keyboard.kicad_pcb (KiCad board)
At the start: 2 copper layers, 331.1 x 102 mm, 150 parts, among them J1 USB_C_Receptacle_USB2.0, Q1 BC858, SW1 SW_Push, SW10 SW_Push, SW11 SW_Push, SW12 SW_Push, SW13 SW_Push, SW14 SW_Push, SW15 SW_Push, SW16 SW_Push, SW17 SW_Push, SW18 SW_Push, SW19 SW_Push, SW2 SW_Push, SW20 SW_Push, SW21 SW_Push, SW22 SW_Push, SW23 SW_Push, SW24 SW_Push, SW25 SW_Push, SW26 SW_Push, SW27 SW_Push, SW28 SW_Push, SW29 SW_Push, SW3 SW_Push, SW30 SW_Push, SW31 SW_Push, SW32 SW_Push, SW33 SW_Push, SW34 SW_Push, SW35 SW_Push, SW36 SW_Push, SW37 SW_Push, SW38 SW_Push, SW39 SW_Push, SW4 SW_Push, SW40 SW_Push, SW41 SW_Push, SW42 SW_Push, SW43 SW_Push, SW44 SW_Push, SW45 SW_Push, SW46 SW_Push, SW47 SW_Push, SW48 SW_Push, SW49 SW_Push, SW5 SW_Push, SW50 SW_Push, SW6 SW_Push, SW7 SW_Push, SW8 SW_Push, SW9 SW_Push, U1 NCP1117-3.3_SOT223, U2 USBLC6-2SC6, U3 W25Q128JVS, U4 RP2040, Y1 ABM8-272_T3

Commit message: Touched up PCB slightly
Routing:
- net GND: vias 36 -> 73
Changed lines of the file:
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@@
     )
   )
+  (gr_circle (center 229.711078 135.3125) (end 229.711078 135.4125)
+    (stroke (width 0.4) (type default)) (fill none) (layer "B.SilkS"))
+  (gr_circle (center 211.461078 108.5625) (end 211.561078 108.5625)
+    (stroke (width 0.3) (type default)) (fill none) (layer "B.SilkS"))
+  (gr_circle (center 217.211078 146.2125) (end 217.311078 146.2125)
+    (stroke (width 0.3) (type default)) (fill none) (layer "B.SilkS"))
   (gr_line locked (start 236.843818 102.346586) (end 252.983253 98.916043)
     (stroke (width 0.2) (type solid)) (layer "Dwgs.User"))
@@
   (via (at 207.711078 140.3125) (size 0.8) (drill 0.4) (layers "F.Cu" "B.Cu") (net 2))
   (via (at 213.961078 155.0625) (size 0.6) (drill 0.35) (layers "F.Cu" "B.Cu") (net 2))
+  (via (at 197.461078 183.8125) (size 0.8) (drill 0.4) (layers "F.Cu" "B.Cu") (free) (net 2))
+  (via (at 197.461078 108.8125) (size 0.8) (drill 0.4) (layers "F.Cu" "B.Cu") (free) (net 2))
+  (via (at 67.461078 123.8125) (size 0.8) (drill 0.4) (layers "F.Cu" "B.Cu") (free) (net 2))
   (via (at 226.961078 117.8125) (size 0.8) (drill 0.4) (layers "F.Cu" "B.Cu") (net 2))
   (via (at 216.716078 106.9125) (size 0.8) (drill 0.4) (layers "F.Cu" "B.Cu") (net 2))
   (via (at 217.75 119) (size 0.8) (drill 0.4) (layers "F.Cu" "B.Cu") (net 2))
+  (via (at 297.461078 123.8125) (size 0.8) (drill 0.4) (layers "F.Cu" "B.Cu") (free) (net 2))
+  (via (at 242.461078 138.8125) (size 0.8) (drill 0.4) (layers "F.Cu" "B.Cu") (free) (net 2))
+  (via (at 242.461078 153.8125) (size 0.8) (drill 0.4) (layers "F.Cu" "B.Cu") (free) (net 2))
+  (via (at 182.461078 183.8125) (size 0.8) (drill 0.4) (layers "F.Cu" "B.Cu") (free) (net 2))
   (via (at 209.711078 132.3125) (size 0.8) (drill 0.4) (layers "F.Cu" "B.Cu") (net 2))
   (via (at 229.75 139.25) (size 0.8) (drill 0.4) (layers "F.Cu" "B.Cu") (net 2))
+  (via (at 107.461078 123.8125) (size 0.8) (drill 0.4) (layers "F.Cu" "B.Cu") (free) (net 2))
+  (via (at 182.461078 123.8125) (size 0.8) (drill 0.4) (layers "F.Cu" "B.Cu") (free) (net 2))
+  (via (at 337.461078 123.8125) (size 0.8) (drill 0.4) (layers "F.Cu" "B.Cu") (free) (net 2))
   (via (at 213.461078 132.3125) (size 0.8) (drill 0.4) (layers "F.Cu" "B.Cu") (net 2))
   (via (at 226.211078 134.3125) (size 0.8) (drill 0.4) (layers "F.Cu" "B.Cu") (net 2))
+  (via (at 197.461078 153.8125) (size 0.8) (drill 0.4) (layers "F.Cu" "B.Cu") (free) (net 2))
+  (via (at 317.461078 123.8125) (size 0.8) (drill 0.4) (layers "F.Cu" "B.Cu") (free) (net 2))
   (via (at 216.966078 110.7125) (size 0.8) (drill 0.4) (layers "F.Cu" "B.Cu") (net 2))
+  (via (at 242.461078 168.8125) (size 0.8) (drill 0.4) (layers "F.Cu" "B.Cu") (free) (net 2))
+  (via (at 372.461078 138.8125) (size 0.8) (drill 0.4) (layers "F.Cu" "B.Cu") (free) (net 2))
+  (via (at 227.461078 108.8125) (size 0.8) (drill 0.4) (layers "F.Cu" "B.Cu") (free) (net 2))
+  (via (at 319.961078 163.8125) (size 0.8) (drill 0.4) (layers "F.Cu" "B.Cu") (free) (net 2))
   (via (at 200.711078 156.0625) (size 0.8) (drill 0.4) (layers "F.Cu" "B.Cu") (net 2))
+  (via (at 227.461078 183.8125) (size 0.8) (drill 0.4) (layers "F.Cu" "B.Cu") (free) (net 2))
   (via (at 215.711078 153.3125) (size 0.8) (drill 0.4) (layers "F.Cu" "B.Cu") (net 2))
+  (via (at 182.461078 138.8125) (size 0.8) (drill 0.4) (layers "F.Cu" "B.Cu") (free) (net 2))
   (via (at 233.461078 116.8125) (size 0.8) (drill 0.4) (layers "F.Cu" "B.Cu") (net 2))
   (via (at 215.711078 157.0625) (size 0.6) (drill 0.35) (layers "F.Cu" "B.Cu") (net 2))
+  (via (at 182.461078 153.8125) (size 0.8) (drill 0.4) (layers "F.Cu" "B.Cu") (free) (net 2))
+  (via (at 212.461078 183.8125) (size 0.8) (drill 0.4) (layers "F.Cu" "B.Cu") (free) (net 2))
+  (via (at 362.461078 88.8125) (size 0.8) (drill 0.4) (layers "F.Cu" "B.Cu") (free) (net 2))
   (via (at 209.711078 140.3125) (size 0.8) (drill 0.4) (layers "F.Cu" "B.Cu") (net 2))
   (via (at 211.211078 156.8125) (size 0.8) (drill 0.4) (layers "F.Cu" "B.Cu") (net 2))
+  (via (at 182.461078 168.8125) (size 0.8) (drill 0.4) (layers "F.Cu" "B.Cu") (free) (net 2))
   (via (at 209.711078 117.3125) (size 0.8) (drill 0.4) (layers "F.Cu" "B.Cu") (net 2))
   (via (at 212.211078 156.3125) (size 0.8) (drill 0.4) (layers "F.Cu" "B.Cu") (net 2))
   (via (at 208.711078 140.3125) (size 0.8) (drill 0.4) (layers "F.Cu" "B.Cu") (net 2))
+  (via (at 52.461078 138.8125) (size 0.8) (drill 0.4) (layers "F.Cu" "B.Cu") (free) (net 2))
   (via (at 207.961078 110.8125) (size 0.8) (drill 0.4) (layers "F.Cu" "B.Cu") (net 2))
+  (via (at 62.461078 88.8125) (size 0.8) (drill 0.4) (layers "F.Cu" "B.Cu") (free) (net 2))
+  (via (at 237.461078 108.8125) (size 0.8) (drill 0.4) (layers "F.Cu" "B.Cu") (free) (net 2))
   (via (at 213.461078 117.3125) (size 0.8) (drill 0.4) (layers "F.Cu" "B.Cu") (net 2))
   (via (at 208.216078 106.9125) (size 0.8) (drill 0.4) (layers "F.Cu" "B.Cu") (net 2))
   (via (at 215.75 120.75) (size 0.8) (drill 0.4) (layers "F.Cu" "B.Cu") (net 2))
   (via (at 207.211078 152.0625) (size 0.8) (drill 0.4) (layers "F.Cu" "B.Cu") (net 2))
+  (via (at 197.461078 103.8125) (size 0.8) (drill 0.4) (layers "F.Cu" "B.Cu") (free) (net 2))
   (via (at 213.211078 158.3125) (size 0.6) (drill 0.35) (layers "F.Cu" "B.Cu") (net 2))
   (via (at 215.711078 110.7125) (size 0.8) (drill 0.4) (layers "F.Cu" "B.Cu") (net 2))
   (via (at 218.961078 144.3125) (size 0.8) (drill 0.4) (layers "F.Cu" "B.Cu") (net 2))
+  (via (at 127.461078 123.8125) (size 0.8) (drill 0.4) (layers "F.Cu" "B.Cu") (free) (net 2))
+  (via (at 102.461078 163.8125) (size 0.8) (drill 0.4) (layers "F.Cu" "B.Cu") (free) (net 2))
+  (via (at 187.461078 108.8125) (size 0.8) (drill 0.4) (layers "F.Cu" "B.Cu") (free) (net 2))
+  (via (at 227.461078 113.8125) (size 0.8) (drill 0.4) (layers "F.Cu" "B.Cu") (free) (net 2))
   (via (at 220.711078 149.5625) (size 0.8) (drill 0.4) (layers "F.Cu" "B.Cu") (net 2))
   (via (at 223.211078 133.25) (size 0.8) (drill 0.4) (layers "F.Cu" "B.Cu") (net 2))
   (via (at 212.461078 108.3125) (size 0.8) (drill 0.4) (layers "F.Cu" "B.Cu") (net 2))
   (via (at 225.211078 124.0625) (size 0.8) (drill 0.4) (layers "F.Cu" "B.Cu") (free) (net 2))
+  (via (at 227.461078 103.8125) (size 0.8) (drill 0.4) (layers "F.Cu" "B.Cu") (free) (net 2))
+  (via (at 87.461078 123.8125) (size 0.8) (drill 0.4) (layers "F.Cu" "B.Cu") (free) (net 2))
   (via (at 207.461078 143.5625) (size 0.8) (drill 0.4) (layers "F.Cu" "B.Cu") (net 2))
+  (via (at 242.461078 123.8125) (size 0.8) (drill 0.4) (layers "F.Cu" "B.Cu") (free) (net 2))
+  (via (at 197.461078 113.8125) (size 0.8) (drill 0.4) (layers "F.Cu" "B.Cu") (free) (net 2))
   (via (at 214.461078 139.5625) (size 0.8) (drill 0.4) (layers "F.Cu" "B.Cu") (net 2))
+  (via (at 357.461078 123.8125) (size 0.8) (drill 0.4) (layers "F.Cu" "B.Cu") (free) (net 2))
+  (via (at 227.461078 153.8125) (size 0.8) (drill 0.4) (layers "F.Cu" "B.Cu") (free) (net 2))
+  (via (at 242.461078 183.8125) (size 0.8) (drill 0.4) (layers "F.Cu" "B.Cu") (free) (net 2))
   (via (at 215.461078 130.0625) (size 0.8) (drill 0.4) (layers "F.Cu" "B.Cu") (net 2))
   (segment (start 209.211078 110.8125) (end 209.211078 109.8225) (width 0.25) (layer "B.Cu") (net 2))

Commit message: PCB ready for production
Parts:
- added ?: LOGO, local-library:rust_crab, F.Cu at (228.2, 164.8)
- ?: renamed from G***; value LOGO -> (none)
- D1: value NCD0805O1 -> NCD0805
- Q1: value BC858 -> S8550
Connections:
- J1 pad S1: unconnected-(J1-SHIELD-PadS1) -> GND
Routing:
- net GND: track 37.7 -> 41.4 mm
Other:
- board text added: "Crab Edition"
