File: pcb/MCU.kicad_sch (KiCad schematic)
At the start: 22 parts, among them U3 RP2040, U4 W25Q128JVS, Y1 ABM8-272_T3

Commit message: Schematic done, starting PCB design
Parts:
- removed R8: DNF, symbol Device:R
- removed R9: 1k, symbol Device:R
- R11: renamed from R5; footprint (none) -> Resistor_SMD:R_0603_1608Metric_Pad0.98x0.95mm_HandSolder
- R12: renamed from R6; footprint (none) -> Resistor_SMD:R_0603_1608Metric_Pad0.98x0.95mm_HandSolder
- R13: renamed from R7; footprint (none) -> Resistor_SMD:R_0603_1608Metric_Pad0.98x0.95mm_HandSolder
- Y1: footprint (none) -> Crystal:Crystal_SMD_3225-4Pin_3.2x2.5mm_HandSoldering
- renumbered C13 to C10, C12 to C11, C11 to C12, C10 to C13, C9 to C14, C8 to C15, C7 to C16, C4 to C3, C3 to C4, C16 to C5, C15 to C6, C5 to C7, C14 to C8, C6 to C9, U4 to U3, U3 to U4
Connections:
- net XIN: now also U4.20 (XIN)
- net XOUT: now also U4.21 (XOUT)
- net row0: now reaches U4.11 (GPIO8)
- net row1: now reaches U4.12 (GPIO9)
- net row2: now reaches U4.13 (GPIO10)
- net row3: now reaches U4.14 (GPIO11)
- net col0: now reaches U4.2 (GPIO0)
- net SWCLK: now reaches U4.24 (SWCLK)
- net SWDIO: now reaches U4.25 (SWD)
- net col1: now reaches U4.3 (GPIO1)
- net col7: now reaches U4.35 (GPIO23)
- net col8: now reaches U4.36 (GPIO24)
- net col9: now reaches U4.37 (GPIO25)
- net col10: now reaches U4.38 (GPIO26_ADC0)
- net col11: now reaches U4.39 (GPIO27_ADC1)
- net col2: now reaches U4.4 (GPIO2)
- net col12: now reaches U4.40 (GPIO28_ADC2)
- net col13: now reaches U4.41 (GPIO29_ADC3)
- net col3: now reaches U4.5 (GPIO3)
- net QSPI_SD3: now reaches U4.51 (QSPI_SD3)
- net QSPI_SD3: now also U3.7 (IO3)
- net QSPI_SCLK: now reaches U4.52 (QSPI_SCLK)
- net QSPI_SCLK: now also U3.6 (CLK)
- net QSPI_SD0: now reaches U4.53 (QSPI_SD0)
- net QSPI_SD0: now also U3.5 (DI(IO0))
- net QSPI_SD2: now reaches U4.54 (QSPI_SD2)
- net QSPI_SD2: now also U3.3 (IO2)
- net QSPI_SD1: now reaches U4.55 (QSPI_SD1)
- net QSPI_SD1: now also U3.2 (DO(IO1))
- net BOOT: now reaches U4.56 (QSPI_SS)
- net BOOT: now also U3.1 (~{CS})
- net col4: now reaches U4.6 (GPIO4)
- net col5: now reaches U4.7 (GPIO5)
- net col6: now reaches U4.8 (GPIO6)
- net USB_D-: now reaches R13.1
- net USB_D+: now reaches R12.1
- no-connect marks 0 -> 12
Other:
- note added: "Flash memory"
- moved on the sheet: C3, C4, C5, R11, U3, Y1

Commit message: Routing in progress
Parts:
- Y1: footprint Crystal:Crystal_SMD_3225-4Pin_3.2x2.5mm_HandSoldering -> Crystal:Crystal_SMD_3225-4Pin_3.2x2.5mm
Connections:
- net col0: now also U4.35 (GPIO23); no longer U4.2 (GPIO0)
- net col1: now also U4.36 (GPIO24); no longer U4.3 (GPIO1)
- net col10: now also U4.5 (GPIO3); no longer U4.38 (GPIO26_ADC0)
- net col11: now also U4.6 (GPIO4); no longer U4.39 (GPIO27_ADC1)
- net col12: now also U4.7 (GPIO5); no longer U4.40 (GPIO28_ADC2)
- net col13: now also U4.8 (GPIO6); no longer U4.41 (GPIO29_ADC3)
- net col2: now also U4.37 (GPIO25); no longer U4.4 (GPIO2)
- net col3: now also U4.38 (GPIO26_ADC0); no longer U4.5 (GPIO3)
- net col4: now also U4.39 (GPIO27_ADC1); no longer U4.6 (GPIO4)
- net col5: now also U4.40 (GPIO28_ADC2); no longer U4.7 (GPIO5)
- net col6: now also U4.41 (GPIO29_ADC3); no longer U4.8 (GPIO6)
- net col7: now also U4.2 (GPIO0); no longer U4.35 (GPIO23)
- net col8: now also U4.3 (GPIO1); no longer U4.36 (GPIO24)
- net col9: now also U4.4 (GPIO2); no longer U4.37 (GPIO25)
Other:
- note added: "Keep C8 close to pin 45"
- note added: "Keep C9 close to pin 44"
- note removed: "Keep C14 close to pin 45"
- note removed: "Keep C6 close to pin 44"

Commit message: More routing progress
Connections:
- net col0: now also U4.41 (GPIO29_ADC3); no longer U4.35 (GPIO23)
- net col1: now also U4.40 (GPIO28_ADC2); no longer U4.36 (GPIO24)
- net col11: now also U4.4 (GPIO2); no longer U4.6 (GPIO4)
- net col12: now also U4.3 (GPIO1); no longer U4.7 (GPIO5)
- net col13: now also U4.2 (GPIO0); no longer U4.8 (GPIO6)
- net col2: now also U4.39 (GPIO27_ADC1); no longer U4.37 (GPIO25)
- net col4: now also U4.37 (GPIO25); no longer U4.39 (GPIO27_ADC1)
- net col5: now also U4.36 (GPIO24); no longer U4.40 (GPIO28_ADC2)
- net col6: now also U4.35 (GPIO23); no longer U4.41 (GPIO29_ADC3)
- net col7: now also U4.8 (GPIO6); no longer U4.2 (GPIO0)
- net col8: now also U4.7 (GPIO5); no longer U4.3 (GPIO1)
- net col9: now also U4.6 (GPIO4); no longer U4.4 (GPIO2)

Commit message: Further progress on routing
Parts:
- added C17: 100n, Capacitor_SMD:C_0603_1608Metric_Pad1.08x0.95mm_HandSolder, symbol Device:C
Connections:
- net +3V3: now also C17.1
- net GND: now also C17.2

Commit message: More routing yippieeeee
Parts:
- removed C16: 100n, Capacitor_SMD:C_0603_1608Metric_Pad1.08x0.95mm_HandSolder, symbol Device:C
- renumbered C17 to C16
Other:
- moved on the sheet: C16
Changed lines of the file:
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@@
   (junction (at 173.99 31.75) (diameter 0) (color 0 0 0 0)
   )
+  (junction (at 168.91 41.91) (diameter 0) (color 0 0 0 0)
+  )
+  (junction (at 237.49 31.75) (diameter 0) (color 0 0 0 0)
+  )
+  (junction (at 158.75 41.91) (diameter 0) (color 0 0 0 0)
+  )
+  (junction (at 207.01 39.37) (diameter 0) (color 0 0 0 0)
+  )
+  (junction (at 196.85 39.37) (diameter 0) (color 0 0 0 0)
+  )
+  (junction (at 177.8 31.75) (diameter 0) (color 0 0 0 0)
+  )
+  (junction (at 217.17 31.75) (diameter 0) (color 0 0 0 0)
+  )
   (junction (at 247.65 39.37) (diameter 0) (color 0 0 0 0)
-  )
-  (junction (at 168.91 41.91) (diameter 0) (color 0 0 0 0)
-  )
-  (junction (at 237.49 31.75) (diameter 0) (color 0 0 0 0)
-  )
-  (junction (at 158.75 41.91) (diameter 0) (color 0 0 0 0)
-  )
-  (junction (at 247.65 31.75) (diameter 0) (color 0 0 0 0)
-  )
-  (junction (at 207.01 39.37) (diameter 0) (color 0 0 0 0)
-  )
-  (junction (at 257.81 39.37) (diameter 0) (color 0 0 0 0)
-  )
-  (junction (at 196.85 39.37) (diameter 0) (color 0 0 0 0)
-  )
-  (junction (at 177.8 31.75) (diameter 0) (color 0 0 0 0)
-  )
-  (junction (at 217.17 31.75) (diameter 0) (color 0 0 0 0)
   )
   (junction (at 29.21 53.34) (diameter 0) (color 0 0 0 0)
@@
     (stroke (width 0) (type default))
   )
-  (wire (pts (xy 257.81 39.37) (xy 247.65 39.37))
-    (stroke (width 0) (type default))
-  )
   (wire (pts (xy 137.16 52.07) (xy 138.43 52.07))
     (stroke (width 0) (type default))
@@
     (stroke (width 0) (type default))
   )
-  (wire (pts (xy 247.65 31.75) (xy 257.81 31.75))
-    (stroke (width 0) (type default))
-  )
   (wire (pts (xy 58.42 83.82) (xy 72.39 83.82))
     (stroke (width 0) (type default))
@@
     (stroke (width 0) (type default))
   )
-  (wire (pts (xy 257.81 39.37) (xy 257.81 40.64))
+  (wire (pts (xy 247.65 39.37) (xy 247.65 40.64))
     (stroke (width 0) (type default))
   )
@@
     )
   )
-  (symbol (lib_id "Device:C") (at 257.81 35.56 0) (unit 1)
-    (in_bom yes) (on_board yes) (dnp no)
-    (property "Reference" "C17" (at 260.35 34.29 0)
-      (effects (font (size 1.27 1.27)) (justify left))
-    )
-    (property "Value" "100n" (at 260.35 36.83 0)
-      (effects (font (size 1.27 1.27)) (justify left))
-    )
-    (property "Footprint" "Capacitor_SMD:C_0603_1608Metric_Pad1.08x0.95mm_HandSolder" (at 258.7752 39.37 0)
-      (effects (font (size 1.27 1.27)) hide)
-    )
-    (property "Datasheet" "~" (at 257.81 35.56 0)
-      (effects (font (size 1.27 1.27)) hide)
-    )
-    (pin "1")
-    (pin "2")
-    (instances
-      (project "keyboard"
-        (path "/fc529d87-72d0-4c92-b352-ddcf4c6f7199/010e79f9-e3f4-42f4-9458-dc603332dc57"
-          (reference "C17") (unit 1)
-        )
-      )
-    )
-  )
-  (symbol (lib_id "power:+1V1") (at 158.75 30.48 0) (unit 1)
-    (in_bom yes) (on_board yes) (dnp no) (fields_autoplaced)
-    (property "Reference" "#PWR018" (at 158.75 34.29 0)
-      (effects (font (size 1.27 1.27)) hide)
-    )
-    (property "Value" "+1V1" (at 158.75 26.67 0)
-      (effects (font (size 1.27 1.27)))
-    )
-    (property "Footprint" "" (at 158.75 30.48 0)
-      (effects (font (size 1.27 1.27)) hide)
-    )
-    (property "Datasheet" "" (at 158.75 30.48 0)
-      (effects (font (size 1.27 1.27)) hide)
-    )
-    (pin "1")
-    (instances
-      (project "keyboard"
-        (path "/fc529d87-72d0-4c92-b352-ddcf4c6f7199/010e79f9-e3f4-42f4-9458-dc603332dc57"
-          (reference "#PWR018") (unit 1)
-        )
-      )
-    )
-  )
-  (symbol (lib_id "power:GND") (at 163.83 135.89 0) (unit 1)
-    (in_bom yes) (on_board yes) (dnp no) (fields_autoplaced)
-    (property "Reference" "#PWR019" (at 163.83 142.24 0)
-      (effects (font (size 1.27 1.27)) hide)
-    )
-    (property "Value" "GND" (at 163.83 140.97 0)
-      (effects (font (size 1.27 1.27)))
-    )
-    (property "Footprint" "" (at 163.83 135.89 0)
-      (effects (font (size 1.27 1.27)) hide)
-    )
-    (property "Datasheet" "" (at 163.83 135.89 0)
-      (effects (font (size 1.27 1.27)) hide)
-    )
-    (pin "1")
-    (instances
-      (project "keyboard"
-        (path "/fc529d87-72d0-4c92-b352-ddcf4c6f7199/010e79f9-e3f4-42f4-9458-dc603332dc57"
-          (reference "#PWR019") (unit 1)
-        )
-      )
-    )
-  )
-  (symbol (lib_id "power:+3V3") (at 137.16 50.8 0) (unit 1)
-    (in_bom yes) (on_board yes) (dnp no) (fields_autoplaced)
-    (property "Reference" "#PWR016" (at 137.16 54.61 0)
-      (effects (font (size 1.27 1.27)) hide)
-    )
-    (property "Value" "+3V3" (at 137.16 46.99 0)
-      (effects (font (size 1.27 1.27)))
-    )
-    (property "Footprint" "" (at 137.16 50.8 0)
-      (effects (font (size 1.27 1.27)) hide)
-    )
-    (property "Datasheet" "" (at 137.16 50.8 0)
-      (effects (font (size 1.27 1.27)) hide)
-    )
-    (pin "1")
-    (instances
-      (project "keyboard"
-        (path "/fc529d87-72d0-4c92-b352-ddcf4c6f7199/010e79f9-e3f4-42f4-9458-dc603332dc57"
-          (reference "#PWR016") (unit 1)
-        )
-      )
-    )
-  )
   (symbol (lib_id "Device:C") (at 247.65 35.56 0) (unit 1)
     (in_bom yes) (on_board yes) (dnp no)
@@
         (path "/fc529d87-72d0-4c92-b352-ddcf4c6f7199/010e79f9-e3f4-42f4-9458-dc603332dc57"
           (reference "C16") (unit 1)
+        )
+      )
+    )
+  )
+  (symbol (lib_id "power:+1V1") (at 158.75 30.48 0) (unit 1)
+    (in_bom yes) (on_board yes) (dnp no) (fields_autoplaced)
+    (property "Reference" "#PWR018" (at 158.75 34.29 0)
+      (effects (font (size 1.27 1.27)) hide)
+    )
+    (property "Value" "+1V1" (at 158.75 26.67 0)
+      (effects (font (size 1.27 1.27)))
+    )
+    (property "Footprint" "" (at 158.75 30.48 0)
+      (effects (font (size 1.27 1.27)) hide)
+    )
+    (property "Datasheet" "" (at 158.75 30.48 0)
+      (effects (font (size 1.27 1.27)) hide)
+    )
+    (pin "1")
+    (instances
+      (project "keyboard"
+        (path "/fc529d87-72d0-4c92-b352-ddcf4c6f7199/010e79f9-e3f4-42f4-9458-dc603332dc57"
+          (reference "#PWR018") (unit 1)
+        )
+      )
+    )
+  )
+  (symbol (lib_id "power:GND") (at 163.83 135.89 0) (unit 1)
+    (in_bom yes) (on_board yes) (dnp no) (fields_autoplaced)
+    (property "Reference" "#PWR019" (at 163.83 142.24 0)
+      (effects (font (size 1.27 1.27)) hide)
+    )
+    (property "Value" "GND" (at 163.83 140.97 0)
+      (effects (font (size 1.27 1.27)))
+    )
+    (property "Footprint" "" (at 163.83 135.89 0)
+      (effects (font (size 1.27 1.27)) hide)
+    )
+    (property "Datasheet" "" (at 163.83 135.89 0)
+      (effects (font (size 1.27 1.27)) hide)
+    )
+    (pin "1")
+    (instances
+      (project "keyboard"
+        (path "/fc529d87-72d0-4c92-b352-ddcf4c6f7199/010e79f9-e3f4-42f4-9458-dc603332dc57"
+          (reference "#PWR019") (unit 1)
+        )
+      )
+    )
+  )
+  (symbol (lib_id "power:+3V3") (at 137.16 50.8 0) (unit 1)
+    (in_bom yes) (on_board yes) (dnp no) (fields_autoplaced)
+    (property "Reference" "#PWR016" (at 137.16 54.61 0)
+      (effects (font (size 1.27 1.27)) hide)
+    )
+    (property "Value" "+3V3" (at 137.16 46.99 0)
+      (effects (font (size 1.27 1.27)))
+    )
+    (property "Footprint" "" (at 137.16 50.8 0)
+      (effects (font (size 1.27 1.27)) hide)
+    )
+    (property "Datasheet" "" (at 137.16 50.8 0)
+      (effects (font (size 1.27 1.27)) hide)
+    )
+    (pin "1")
+    (instances
+      (project "keyboard"
+        (path "/fc529d87-72d0-4c92-b352-ddcf4c6f7199/010e79f9-e3f4-42f4-9458-dc603332dc57"
+          (reference "#PWR016") (unit 1)
         )
       )
@@
     )
   )
-  (symbol (lib_id "power:GND") (at 257.81 40.64 0) (unit 1)
-    (in_bom yes) (on_board yes) (dnp no) (fields_autoplaced)
-    (property "Reference" "#PWR021" (at 257.81 46.99 0)
-      (effects (font (size 1.27 1.27)) hide)
-    )
-    (property "Value" "GND" (at 257.81 45.72 0)
-      (effects (font (size 1.27 1.27)))
-    )
-    (property "Footprint" "" (at 257.81 40.64 0)
-      (effects (font (size 1.27 1.27)) hide)
-    )
-    (property "Datasheet" "" (at 257.81 40.64 0)
-      (effects (font (size 1.27 1.27)) hide)
-    )
+  (symbol (lib_id "power:GND") (at 247.65 40.64 0) (unit 1)
+    (in_bom yes) (on_board yes) (dnp no) (fields_autoplaced)
+    (property "Reference" "#PWR021" (at 247.65 46.99 0)
+      (effects (font (size 1.27 1.27)) hide)
+    )
+    (property "Value" "GND" (at 247.65 45.72 0)
+      (effects (font (size 1.27 1.27)))
+    )
+    (property "Footprint" "" (at 247.65 40.64 0)
+      (effects (font (size 1.27 1.27)) hide)
+    )
+    (property "Datasheet" "" (at 247.65 40.64 0)
+      (effects (font (size 1.27 1.27)) hide)
+    )

Commit message: Rerouted a lot of stuff
Parts:
- removed C16: 100n, Capacitor_SMD:C_0603_1608Metric_Pad1.08x0.95mm_HandSolder, symbol Device:C
- added C2: 100n, Capacitor_SMD:C_0402_1005Metric, symbol Device:C
- C10, C11, C12, C13, C14, C15, C5, C6, C7, C8, C9: footprint Capacitor_SMD:C_0603_1608Metric_Pad1.08x0.95mm_HandSolder -> Capacitor_SMD:C_0402_1005Metric
- C3, C4: footprint Capacitor_SMD:C_0805_2012Metric_Pad1.18x1.45mm_HandSolder -> Capacitor_SMD:C_0402_1005Metric
- R11, R12, R13: footprint Resistor_SMD:R_0603_1608Metric_Pad0.98x0.95mm_HandSolder -> Resistor_SMD:R_0402_1005Metric
Connections:
- net +1V1: now also C2.1; no longer C7.1
- net +3V3: now also C7.1
- net GND: now also C4.2, C2.2; no longer C4.1
- net at R11.1, Y1.3: now also C4.1; no longer C4.2

Commit message: PCB design complete
Parts:
- C10, C11, C12, C13, C14, C15, C2, C5, C6, C7: LCSC (none) -> C1525
- C3, C4: LCSC (none) -> C1548
- R11: LCSC (none) -> C11702
- R12, R13: LCSC (none) -> C25100
- U3: LCSC (none) -> C97521
- U4: LCSC (none) -> C2040
- Y1: LCSC (none) -> C20625731
Changed lines of the file:
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@@
     (stroke (width 0) (type default))
   )
-  (wire (pts (xy 54.61 48.26) (xy 57.15 48.26))
+  (wire (pts (xy 54.61 48.26) (xy 55.88 48.26))
     (stroke (width 0) (type default))
   )
@@
       (effects (font (size 1.27 1.27)) hide)
     )
+    (property "LCSC" "C20625731" (at 49.53 48.26 90)
+      (effects (font (size 1.27 1.27)) hide)
+    )
     (pin "1")
     (pin "2")
@@
     )
     (property "Datasheet" "https://datasheets.raspberrypi.com/rp2040/rp2040-datasheet.pdf" (at 163.83 90.17 0)
+      (effects (font (size 1.27 1.27)) hide)
+    )
+    (property "LCSC" "C2040" (at 163.83 90.17 0)
       (effects (font (size 1.27 1.27)) hide)
     )
@@
       (effects (font (size 1.27 1.27)) hide)
     )
+    (property "LCSC" "C1525" (at 72.39 88.9 0)
+      (effects (font (size 1.27 1.27)) hide)
+    )
     (pin "1")
     (pin "2")
@@
       (effects (font (size 1.27 1.27)) hide)
     )
+    (property "LCSC" "C1525" (at 186.69 35.56 0)
+      (effects (font (size 1.27 1.27)) hide)
+    )
     (pin "1")
     (pin "2")
@@
       (effects (font (size 1.27 1.27)) hide)
     )
+    (property "LCSC" "C1525" (at 217.17 35.56 0)
+      (effects (font (size 1.27 1.27)) hide)
+    )
     (pin "1")
     (pin "2")
@@
       (effects (font (size 1.27 1.27)) hide)
     )
-    (property "Value" "GND" (at 39.37 49.53 0)
+    (property "Value" "GND" (at 43.18 52.07 0)
       (effects (font (size 1.27 1.27)))
     )
@@
       (effects (font (size 1.27 1.27)) hide)
     )
+    (property "LCSC" "C1525" (at 140.97 35.56 0)
+      (effects (font (size 1.27 1.27)) hide)
+    )
     (pin "1")
     (pin "2")
@@
     )
     (property "Datasheet" "~" (at 67.31 53.34 0)
+      (effects (font (size 1.27 1.27)) hide)
+    )
+    (property "LCSC" "C11702" (at 67.31 53.34 90)
       (effects (font (size 1.27 1.27)) hide)
     )
@@
       (effects (font (size 1.27 1.27)) hide)
     )
+    (property "LCSC" "C1525" (at 207.01 35.56 0)
+      (effects (font (size 1.27 1.27)) hide)
+    )
     (pin "1")
     (pin "2")
@@
       (effects (font (size 1.27 1.27)) hide)
     )
+    (property "LCSC" "C1525" (at 237.49 35.56 0)
+      (effects (font (size 1.27 1.27)) hide)
+    )
     (pin "1")
     (pin "2")
@@
       (effects (font (size 1.27 1.27)) hide)
     )
+    (property "LCSC" "C1525" (at 247.65 35.56 0)
+      (effects (font (size 1.27 1.27)) hide)
+    )
     (pin "1")
     (pin "2")
@@
       (effects (font (size 1.27 1.27)) hide)
     )
+    (property "LCSC" "C1525" (at 227.33 35.56 0)
+      (effects (font (size 1.27 1.27)) hide)
+    )
     (pin "1")
     (pin "2")
@@
     )
     (property "Datasheet" "http://www.winbond.com/resource-files/w25q128jv_dtr%20revc%2003272018%20plus.pdf" (at 58.42 101.6 0)
+      (effects (font (size 1.27 1.27)) hide)
+    )
+    (property "LCSC" "C97521" (at 58.42 101.6 0)
       (effects (font (size 1.27 1.27)) hide)
     )
@@
       (effects (font (size 1.27 1.27)) hide)
     )
+    (property "LCSC" "C25100" (at 127 57.15 90)
+      (effects (font (size 1.27 1.27)) hide)
+    )
     (pin "1")
     (pin "2")
@@
       (effects (font (size 1.27 1.27)) hide)
     )
+    (property "LCSC" "C1525" (at 130.81 35.56 0)
+      (effects (font (size 1.27 1.27)) hide)
+    )
     (pin "1")
     (pin "2")
@@
       (effects (font (size 1.27 1.27)) hide)
     )
+    (property "LCSC" "C1525" (at 196.85 35.56 0)
+      (effects (font (size 1.27 1.27)) hide)
+    )
     (pin "1")
     (pin "2")
@@
       (effects (font (size 1.27 1.27)) hide)
     )
+    (property "LCSC" "C25100" (at 127 64.77 90)
+      (effects (font (size 1.27 1.27)) hide)
+    )
     (pin "1")
     (pin "2")
@@
     )
   )
-  (symbol (lib_id "power:GND") (at 57.15 48.26 0) (unit 1)
-    (in_bom yes) (on_board yes) (dnp no)
-    (property "Reference" "#PWR06" (at 57.15 54.61 0)
-      (effects (font (size 1.27 1.27)) hide)
-    )
-    (property "Value" "GND" (at 60.96 49.53 0)
-      (effects (font (size 1.27 1.27)))
-    )
-    (property "Footprint" "" (at 57.15 48.26 0)
-      (effects (font (size 1.27 1.27)) hide)
-    )
-    (property "Datasheet" "" (at 57.15 48.26 0)
+  (symbol (lib_id "power:GND") (at 55.88 48.26 0) (unit 1)
+    (in_bom yes) (on_board yes) (dnp no)
+    (property "Reference" "#PWR06" (at 55.88 54.61 0)
+      (effects (font (size 1.27 1.27)) hide)
+    )
+    (property "Value" "GND" (at 55.88 52.07 0)
+      (effects (font (size 1.27 1.27)))
+    )
+    (property "Footprint" "" (at 55.88 48.26 0)
+      (effects (font (size 1.27 1.27)) hide)
+    )
+    (property "Datasheet" "" (at 55.88 48.26 0)
       (effects (font (size 1.27 1.27)) hide)
     )
@@
       (effects (font (size 1.27 1.27)) hide)
     )
+    (property "LCSC" "C1548" (at 35.56 43.18 0)
+      (effects (font (size 1.27 1.27)) hide)
+    )
     (pin "1")
     (pin "2")
@@
       (effects (font (size 1.27 1.27)) hide)
     )
+    (property "LCSC" "C1548" (at 35.56 53.34 0)
+      (effects (font (size 1.27 1.27)) hide)
+    )
