File: pcb/MCU.kicad_sch (KiCad schematic)
At the start: 20 parts, among them U3 W25Q128JVS, U4 RP2040, Y1 ABM8-272_T3

Commit message: PCB ready for production
Parts:
- C8, C9: LCSC (none) -> C52923
Changed lines of the file:
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@@
+      (effects (font (size 1.27 1.27)) hide)
+    )
+    (property "LCSC" "C52923" (at 151.13 35.56 0)
       (effects (font (size 1.27 1.27)) hide)
     )
@@
       (effects (font (size 1.27 1.27)) hide)
     )
+    (property "LCSC" "C52923" (at 177.8 35.56 0)
+      (effects (font (size 1.27 1.27)) hide)
+    )
